File: MacroX4.kicad_sch (KiCad schematic)
At the start: 49 parts, among them J1 S2B-PH-K-S_LF__SN_, SW1 RotaryEncoder_Switch, SW2 RotaryEncoder_Switch, U1 Nice_Nano_V2

Commit message: Wiring and more components
Parts:
- added SW3: 1825910-6, 1825910-6:SW_1825910-6-4, symbol 1825910-6:1825910-6
Connections:
- net Column 4: now also S10.1, S5.1, SW1.S2, SW2.S2
- net Ground 1: now also SW3.4
- net Row 2: now also D17.1 (K)
- net Reset: now reaches U1.22 (RST)
- net Reset: now also SW3.1
Changed lines of the file:
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@@
   (junction (at 68.58 88.9) (diameter 0) (color 0 0 0 0)
   )
+  (junction (at 50.8 76.2) (diameter 0) (color 0 0 0 0)
+  )
+  (junction (at 76.2 76.2) (diameter 0) (color 0 0 0 0)
+  )
+  (junction (at 50.8 101.6) (diameter 0) (color 0 0 0 0)
+  )
+  (junction (at 81.28 114.3) (diameter 0) (color 0 0 0 0)
+  )
+  (junction (at 81.28 88.9) (diameter 0) (color 0 0 0 0)
+  )
+  (junction (at 55.88 114.3) (diameter 0) (color 0 0 0 0)
+  )
+  (junction (at 93.98 139.7) (diameter 0) (color 0 0 0 0)
+  )
+  (junction (at 93.98 63.5) (diameter 0) (color 0 0 0 0)
+  )
+  (junction (at 68.58 139.7) (diameter 0) (color 0 0 0 0)
+  )
+  (junction (at 76.2 50.8) (diameter 0) (color 0 0 0 0)
+  )
+  (junction (at 63.5 76.2) (diameter 0) (color 0 0 0 0)
+  )
+  (junction (at 88.9 50.8) (diameter 0) (color 0 0 0 0)
+  )
+  (junction (at 63.5 101.6) (diameter 0) (color 0 0 0 0)
+  )
   (junction (at 101.6 76.2) (diameter 0) (color 0 0 0 0)
   )
-  (junction (at 50.8 76.2) (diameter 0) (color 0 0 0 0)
-  )
-  (junction (at 76.2 76.2) (diameter 0) (color 0 0 0 0)
-  )
-  (junction (at 50.8 101.6) (diameter 0) (color 0 0 0 0)
-  )
-  (junction (at 81.28 114.3) (diameter 0) (color 0 0 0 0)
-  )
-  (junction (at 81.28 88.9) (diameter 0) (color 0 0 0 0)
-  )
-  (junction (at 55.88 114.3) (diameter 0) (color 0 0 0 0)
-  )
-  (junction (at 93.98 139.7) (diameter 0) (color 0 0 0 0)
-  )
-  (junction (at 93.98 63.5) (diameter 0) (color 0 0 0 0)
-  )
-  (junction (at 68.58 139.7) (diameter 0) (color 0 0 0 0)
-  )
-  (junction (at 76.2 50.8) (diameter 0) (color 0 0 0 0)
-  )
-  (junction (at 63.5 76.2) (diameter 0) (color 0 0 0 0)
-  )
-  (junction (at 88.9 50.8) (diameter 0) (color 0 0 0 0)
-  )
-  (junction (at 63.5 101.6) (diameter 0) (color 0 0 0 0)
-  )
-  (junction (at 106.68 114.3) (diameter 0) (color 0 0 0 0)
-  )
   (junction (at 55.88 139.7) (diameter 0) (color 0 0 0 0)
   )
@@
   (junction (at 50.8 50.8) (diameter 0) (color 0 0 0 0)
   )
-  (junction (at 106.68 101.6) (diameter 0) (color 0 0 0 0)
+  (junction (at 101.6 50.8) (diameter 0) (color 0 0 0 0)
   )
   (junction (at 88.9 101.6) (diameter 0) (color 0 0 0 0)
@@
   (junction (at 88.9 76.2) (diameter 0) (color 0 0 0 0)
   )
+  (junction (at 115.57 91.44) (diameter 0) (color 0 0 0 0)
+  )
+  (junction (at 93.98 114.3) (diameter 0) (color 0 0 0 0)
+  )
   (junction (at 93.98 88.9) (diameter 0) (color 0 0 0 0)
   )
@@
     (stroke (width 0) (type default))
   )
-  (wire (pts (xy 106.68 114.3) (xy 114.3 114.3))
-    (stroke (width 0) (type default))
-  )
   (wire (pts (xy 40.64 88.9) (xy 55.88 88.9))
     (stroke (width 0) (type default))
@@
     (stroke (width 0) (type default))
   )
+  (wire (pts (xy 115.57 76.2) (xy 115.57 91.44))
+    (stroke (width 0) (type default))
+  )
   (wire (pts (xy 81.28 139.7) (xy 93.98 139.7))
     (stroke (width 0) (type default))
   )
+  (wire (pts (xy 109.22 116.84) (xy 144.78 116.84))
+    (stroke (width 0) (type default))
+  )
   (wire (pts (xy 88.9 43.18) (xy 88.9 50.8))
     (stroke (width 0) (type default))
@@
     (stroke (width 0) (type default))
   )
+  (wire (pts (xy 109.22 127) (xy 114.3 127))
+    (stroke (width 0) (type default))
+  )
   (wire (pts (xy 88.9 101.6) (xy 88.9 127))
     (stroke (width 0) (type default))
@@
     (stroke (width 0) (type default))
   )
+  (wire (pts (xy 144.78 91.44) (xy 144.78 116.84))
+    (stroke (width 0) (type default))
+  )
   (wire (pts (xy 81.28 63.5) (xy 93.98 63.5))
     (stroke (width 0) (type default))
@@
     (stroke (width 0) (type default))
   )
-  (wire (pts (xy 106.68 127) (xy 114.3 127))
+  (wire (pts (xy 101.6 43.18) (xy 101.6 50.8))
+    (stroke (width 0) (type default))
+  )
+  (wire (pts (xy 106.68 101.6) (xy 114.3 101.6))
     (stroke (width 0) (type default))
   )
@@
     (stroke (width 0) (type default))
   )
-  (wire (pts (xy 106.68 114.3) (xy 106.68 127))
-    (stroke (width 0) (type default))
-  )
   (wire (pts (xy 93.98 63.5) (xy 106.68 63.5))
     (stroke (width 0) (type default))
   )
-  (wire (pts (xy 101.6 76.2) (xy 101.6 93.98))
-    (stroke (width 0) (type default))
-  )
   (wire (pts (xy 63.5 50.8) (xy 63.5 76.2))
     (stroke (width 0) (type default))
@@
     (stroke (width 0) (type default))
   )
+  (wire (pts (xy 106.68 91.44) (xy 115.57 91.44))
+    (stroke (width 0) (type default))
+  )
   (wire (pts (xy 154.94 76.2) (xy 176.53 76.2))
     (stroke (width 0) (type default))
@@
     (stroke (width 0) (type default))
   )
+  (wire (pts (xy 106.68 91.44) (xy 106.68 101.6))
+    (stroke (width 0) (type default))
+  )
   (wire (pts (xy 55.88 139.7) (xy 68.58 139.7))
     (stroke (width 0) (type default))
@@
     (stroke (width 0) (type default))
   )
-  (wire (pts (xy 106.68 99.06) (xy 106.68 101.6))
+  (wire (pts (xy 109.22 116.84) (xy 109.22 127))
+    (stroke (width 0) (type default))
+  )
+  (wire (pts (xy 93.98 114.3) (xy 114.3 114.3))
+    (stroke (width 0) (type default))
+  )
+  (wire (pts (xy 115.57 91.44) (xy 144.78 91.44))
     (stroke (width 0) (type default))
   )
@@
     (stroke (width 0) (type default))
   )
-  (wire (pts (xy 106.68 101.6) (xy 106.68 114.3))
-    (stroke (width 0) (type default))
-  )
   (wire (pts (xy 55.88 114.3) (xy 68.58 114.3))
     (stroke (width 0) (type default))
   )
-  (wire (pts (xy 101.6 93.98) (xy 106.68 99.06))
+  (wire (pts (xy 101.6 76.2) (xy 115.57 76.2))
     (stroke (width 0) (type default))
   )
@@
     (stroke (width 0) (type default))
   )
-  (wire (pts (xy 106.68 101.6) (xy 114.3 101.6))
-    (stroke (width 0) (type default))
-  )
   (global_label "Ground 3" (shape input) (at 241.3 43.18 270) (fields_autoplaced)
     (effects (font (size 1.27 1.27)) (justify right))
@@
     )
   )
+  (global_label "Ground 1" (shape input) (at 193.04 109.22 0) (fields_autoplaced)
+    (effects (font (size 1.27 1.27)) (justify left))
+    (property "Intersheetrefs" "${INTERSHEET_REFS}" (at 204.8545 109.22 0)
+      (effects (font (size 1.27 1.27)) (justify left) hide)
+    )
+  )
   (global_label "Negative" (shape input) (at 151.13 31.75 180) (fields_autoplaced)
     (effects (font (size 1.27 1.27)) (justify right))
@@
     )
   )
+  (global_label "Reset" (shape input) (at 181.61 36.83 0) (fields_autoplaced)
+    (effects (font (size 1.27 1.27)) (justify left))
+    (property "Intersheetrefs" "${INTERSHEET_REFS}" (at 189.7962 36.83 0)
+      (effects (font (size 1.27 1.27)) (justify left) hide)
+    )
+  )
   (global_label "Column 4" (shape input) (at 101.6 43.18 90) (fields_autoplaced)
     (effects (font (size 1.27 1.27)) (justify left))
@@
     (effects (font (size 1.27 1.27)) (justify right))
     (property "Intersheetrefs" "${INTERSHEET_REFS}" (at 225.0706 35.56 0)
+      (effects (font (size 1.27 1.27)) (justify right) hide)
+    )
+  )
+  (global_label "Reset" (shape input) (at 172.72 104.14 180) (fields_autoplaced)
+    (effects (font (size 1.27 1.27)) (justify right))
+    (property "Intersheetrefs" "${INTERSHEET_REFS}" (at 164.5338 104.14 0)
       (effects (font (size 1.27 1.27)) (justify right) hide)
     )
@@
         )
       )
+    )
+  )
+  (symbol (lib_id "1825910-6:1825910-6") (at 182.88 106.68 0) (unit 1)
+    (in_bom yes) (on_board yes) (dnp no) (fields_autoplaced)
+    (property "Reference" "SW3" (at 182.88 96.52 0)
+      (effects (font (size 1.27 1.27)))
+    )
+    (property "Value" "1825910-6" (at 182.88 99.06 0)
+      (effects (font (size 1.27 1.27)))
+    )
+    (property "Footprint" "1825910-6:SW_1825910-6-4" (at 182.88 106.68 0)
+      (effects (font (size 1.27 1.27)) (justify bottom) hide)
+    )
+    (property "Datasheet" "" (at 182.88 106.68 0)
+      (effects (font (size 1.27 1.27)) hide)
+    )
+    (property "Comment" "1825910-6" (at 182.88 106.68 0)
+      (effects (font (size 1.27 1.27)) (justify bottom) hide)
+    )
+    (property "MF" "TE Connectivity" (at 182.88 106.68 0)
+      (effects (font (size 1.27 1.27)) (justify bottom) hide)
+    )
+    (property "Description" "\nSwitch Push Button OFF (ON) SPST Round Button 0.05A 24VDC Momentary Contact PC Pins Thru-Hole\n" (at 182.88 106.68 0)
+      (effects (font (size 1.27 1.27)) (justify bottom) hide)
+    )
+    (property "Package" "None" (at 182.88 106.68 0)
+      (effects (font (size 1.27 1.27)) (justify bottom) hide)
+    )
+    (property "Price" "None" (at 182.88 106.68 0)
+      (effects (font (size 1.27 1.27)) (justify bottom) hide)
+    )
+    (property "Check_prices" "https://www.snapeda.com/parts/1825910-6/TE+Connectivity+ALCOSWITCH+Switches/view-part/?ref=eda" (at 182.88 106.68 0)
+      (effects (font (size 1.27 1.27)) (justify bottom) hide)
+    )
+    (property "STANDARD" "Manufacturer Recommendations" (at 182.88 106.68 0)
+      (effects (font (size 1.27 1.27)) (justify bottom) hide)
+    )
+    (property "PARTREV" "C10" (at 182.88 106.68 0)
+      (effects (font (size 1.27 1.27)) (justify bottom) hide)
+    )
+    (property "SnapEDA_Link" "https://www.snapeda.com/parts/1825910-6/TE+Connectivity+ALCOSWITCH+Switches/view-part/?ref=snap" (at 182.88 106.68 0)
+      (effects (font (size 1.27 1.27)) (justify bottom) hide)
+    )
+    (property "MP" "1825910-6" (at 182.88 106.68 0)
+      (effects (font (size 1.27 1.27)) (justify bottom) hide)
+    )
+    (property "Purchase-URL" "https://www.snapeda.com/api/url_track_click_mouser/?unipart_id=226996&manufacturer=TE Connectivity&part_name=1825910-6&search_term=None" (at 182.88 106.68 0)
+      (effects (font (size 1.27 1.27)) (justify bottom) hide)
+    )
+    (property "Availability" "In Stock" (at 182.88 106.68 0)
+      (effects (font (size 1.27 1.27)) (justify bottom) hide)
+    )
+    (property "MANUFACTURER" "TE CONNECTIVITY" (at 182.88 106.68 0)
+      (effects (font (size 1.27 1.27)) (justify bottom) hide)
+    )
+    (pin "1")
+    (pin "3")
+    (pin "2")
+    (pin "4")
+    (instances
+      (project "MacroX4"
+        (path "/c660ade3-d089-4c43-b966-0b98c189f05e"
+          (reference "SW3") (unit 1)
+        )
+      )
